File: etapa_3/PCB/Modulo_corrente_temperatura_barco_Zenite-V02/Modulo_corrente_temperatura_barco_Zenite.kicad_sch (KiCad schematic)
At the start: 47 parts, among them J1 RJ45_Shielded, J2 RJ45_Shielded, J3 Conn_01x03, U2 LM7805, U3 TLV2376IDGKR, U4 MCP2515-xSO, U5 MCP2551-I-SN, Y1 16MHz

Commit message: minor ajustmentes in PCB laytout and schem
Parts:
- removed J3: Conn_01x03, pi-III-lib:B3BXHALFSN, symbol Connector_Generic:Conn_01x03
- added J3: 2edgrc, pi-III-lib:2EDRC_4pins, symbol Connector_Generic:Conn_01x04
- R14, R8: footprint Resistor_SMD:R_2010_5025Metric_Pad1.40x2.65mm_HandSolder -> Resistor_SMD:R_1206_3216Metric_Pad1.30x1.75mm_HandSolder
Connections:
- net 12V: now also J3.2 (Pin_2)
- net I_signal: now also J3.3 (Pin_3)
- net neg12V: now also J3.1 (Pin_1)
- no-connect marks 31 -> 32
Changed lines of the file:
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@@
 	)
 	(no_connect
+		(at 99.06 26.67)
+	)
+	(no_connect
 		(at 133.35 168.91)
 	)
@@
 	(wire
 		(pts
+			(xy 97.79 19.05) (xy 99.06 19.05)
+		)
+		(stroke
+			(width 0)
+			(type default)
+		)
+	)
+	(wire
+		(pts
 			(xy 40.64 91.44) (xy 41.91 91.44)
 		)
@@
 	(wire
 		(pts
-			(xy 97.79 26.67) (xy 99.06 26.67)
-		)
-		(stroke
-			(width 0)
-			(type default)
-		)
-	)
-	(wire
-		(pts
 			(xy 172.72 38.1) (xy 173.99 38.1)
 		)
@@
 		)
 	)
-	(global_label "NSS2"
+	(global_label "neg12V"
 		(shape input)
-		(at 31.75 140.97 180)
+		(at 97.79 19.05 180)
 		(fields_autoplaced yes)
 		(effects
@@
 		)
 		(property "Intersheetrefs" "${INTERSHEET_REFS}"
-			(at 23.8058 140.97 0)
+			(at 87.9106 19.05 0)
 			(effects
 				(font
@@
 		)
 	)
-	(global_label "A10"
+	(global_label "NSS2"
 		(shape input)
-		(at 31.75 156.21 180)
+		(at 31.75 140.97 180)
 		(fields_autoplaced yes)
 		(effects
@@
 		)
 		(property "Intersheetrefs" "${INTERSHEET_REFS}"
-			(at 25.2572 156.21 0)
+			(at 23.8058 140.97 0)
 			(effects
 				(font
@@
 		)
 	)
-	(global_label "CAN_18V"
+	(global_label "A10"
 		(shape input)
-		(at 64.77 33.02 180)
+		(at 31.75 156.21 180)
 		(fields_autoplaced yes)
 		(effects
@@
 		)
 		(property "Intersheetrefs" "${INTERSHEET_REFS}"
-			(at 53.6205 33.02 0)
+			(at 25.2572 156.21 0)
 			(effects
 				(font
@@
 	(global_label "CAN_18V"
 		(shape input)
-		(at 148.59 20.32 180)
+		(at 64.77 33.02 180)
 		(fields_autoplaced yes)
 		(effects
@@
 		)
 		(property "Intersheetrefs" "${INTERSHEET_REFS}"
-			(at 137.4405 20.32 0)
+			(at 53.6205 33.02 0)
 			(effects
 				(font
@@
 		)
 	)
-	(global_label "12V"
+	(global_label "CAN_18V"
 		(shape input)
-		(at 199.39 36.83 180)
+		(at 148.59 20.32 180)
 		(fields_autoplaced yes)
 		(effects
@@
 		)
 		(property "Intersheetrefs" "${INTERSHEET_REFS}"
-			(at 192.8972 36.83 0)
+			(at 137.4405 20.32 0)
 			(effects
 				(font
@@
 		)
 	)
-	(global_label "neg12V"
+	(global_label "12V"
 		(shape input)
-		(at 97.79 26.67 180)
+		(at 199.39 36.83 180)
 		(fields_autoplaced yes)
 		(effects
@@
 		)
 		(property "Intersheetrefs" "${INTERSHEET_REFS}"
-			(at 87.9106 26.67 0)
+			(at 192.8972 36.83 0)
 			(effects
 				(font
@@
 	)
 	(symbol
+		(lib_id "Connector_Generic:Conn_01x04")
+		(at 104.14 21.59 0)
+		(unit 1)
+		(exclude_from_sim no)
+		(in_bom yes)
+		(on_board yes)
+		(dnp no)
+		(property "Reference" "J3"
+			(at 106.68 21.5899 0)
+			(effects
+				(font
+					(size 1.27 1.27)
+				)
+				(justify left)
+			)
+		)
+		(property "Value" "2edgrc"
+			(at 99.06 29.21 0)
+			(effects
+				(font
+					(size 1.27 1.27)
+				)
+				(justify left)
+			)
+		)
+		(property "Footprint" "pi-III-lib:2EDRC_4pins"
+			(at 104.14 21.59 0)
+			(effects
+				(font
+					(size 1.27 1.27)
+				)
+				(hide yes)
+			)
+		)
+		(property "Datasheet" "~"
+			(at 104.14 21.59 0)
+			(effects
+				(font
+					(size 1.27 1.27)
+				)
+				(hide yes)
+			)
+		)
+		(property "Description" "Generic connector, single row, 01x04, script generated (kicad-library-utils/schlib/autogen/connector/)"
+			(at 104.14 21.59 0)
+			(effects
+				(font
+					(size 1.27 1.27)
+				)
+				(hide yes)
+			)
+		)
+		(pin "1"
+		)
+		(pin "3"
+		)
+		(pin "4"
+		)
+		(pin "2"
+		)
+		(instances
+			(project ""
+				(path "/1b5e2233-3864-4906-b770-4c3dd25f47ba"
+					(reference "J3")
+					(unit 1)
+				)
+			)
+		)
+	)
+	(symbol
 		(lib_id "Device:R")
 		(at 215.9 121.92 0)
@@
 	)
 	(symbol
-		(lib_id "Connector_Generic:Conn_01x03")
-		(at 104.14 24.13 0)
-		(unit 1)
-		(exclude_from_sim no)
-		(in_bom yes)
-		(on_board yes)
-		(dnp no)
-		(property "Reference" "J3"
-			(at 102.87 15.24 0)
-			(effects
-				(font
-					(size 1.27 1.27)
-				)
-				(justify left)
-			)
-		)
-		(property "Value" "Conn_01x03"
-			(at 99.06 17.78 0)
-			(effects
-				(font
-					(size 1.27 1.27)
-				)
-				(justify left)
-			)
-		)
-		(property "Footprint" "pi-III-lib:B3BXHALFSN"
-			(at 104.14 24.13 0)
-			(effects
-				(font
-					(size 1.27 1.27)
-				)
-				(hide yes)
-			)
-		)
-		(property "Datasheet" "~"
-			(at 104.14 24.13 0)
-			(effects
-				(font
-					(size 1.27 1.27)
-				)
-				(hide yes)
-			)
-		)
-		(property "Description" "Generic connector, single row, 01x03, script generated (kicad-library-utils/schlib/autogen/connector/)"
-			(at 104.14 24.13 0)
-			(effects
-				(font
-					(size 1.27 1.27)
-				)
-				(hide yes)
-			)
-		)
-		(pin "1"
-		)
-		(pin "3"
-		)
-		(pin "2"
-		)
-		(instances
-			(project ""
-				(path "/1b5e2233-3864-4906-b770-4c3dd25f47ba"
-					(reference "J3")
-					(unit 1)
-				)
-			)
-		)
-	)
-	(symbol
 		(lib_id "power:GND")
 		(at 57.15 123.19 0)
@@
 			)
 		)
-		(property "Footprint" "Resistor_SMD:R_2010_5025Metric_Pad1.40x2.65mm_HandSolder"
+		(property "Footprint" "Resistor_SMD:R_1206_3216Metric_Pad1.30x1.75mm_HandSolder"
 			(at 192.532 121.92 90)
 			(effects
@@
 			)
 		)
-		(property "Footprint" "Resistor_SMD:R_2010_5025Metric_Pad1.40x2.65mm_HandSolder"
+		(property "Footprint" "Resistor_SMD:R_1206_3216Metric_Pad1.30x1.75mm_HandSolder"
 			(at 198.882 121.92 90)
 			(effects
