File: etapa_3/PCB/Modulo_corrente_temperatura_barco_Zenite-V02/Modulo_corrente_temperatura_barco_Zenite.kicad_pcb (KiCad board)
At the start: 2 copper layers, 60 x 138.6 mm, 47 parts, among them J1 RJ45_Shielded, J2 RJ45_Shielded, J3 2edgrc, U2 LM7805, U3 TLV2376IDGKR, U4 MCP2515-xSO, U5 MCP2551-I-SN, Y1 16MHz

Commit message: Etapa 3 documentation update
Parts:
- moved C9 0.06 mm to (133.4, 57.5)
- moved C10 0.05 mm to (137.2, 57.5)
Routing:
- net GND: track 54.3 -> 566.7 mm, vias 17 -> 16
- net AGND: track 2.79 -> 14.9 mm
- removed copper zone on F.Cu, net GND
